Commit message: changed file locations from /home/simon to ./ in arm_test_time and robot_obj_combined_hulls

File: lsa1.1_new/robot_obj_combined_hulls.urdf (robot description, URDF)
Before this commit: robot LSA, 146 links, 145 joints
Links:
- link column_link: geometry collision mesh filename=./lsa1.1_new//meshes/urdf/obj_combined_hulls/column_link.obj; visual mesh filename=./lsa1.1_new//meshes/urdf/obj_combined_hulls/column_link.obj
- link hydraulic_container_link: geometry collision mesh filename=./lsa1.1_new//meshes/urdf/obj_combined_hulls/hydraulic_cont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; visual mesh filename=./lsa1.1_new//meshes/urdf/obj_combined_hulls/hydraulic_cont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
- link left_caster_link: geometry collision mesh filename=./lsa1.1_new//meshes/urdf/obj_combined_hulls/left_caster_li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; visual mesh filename=./lsa1.1_new//meshes/urdf/obj_combined_hulls/left_caster_li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
- link left_caster_swivel_link: geometry collision mesh filename=./lsa1.1_new//meshes/urdf/obj_combined_hulls/left_caster_sw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; visual mesh filename=./lsa1.1_new//meshes/urdf/obj_combined_hulls/left_caster_sw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
- link left_elbow_fe_link: geometry collision mesh filename=./lsa1.1_new//meshes/urdf/obj_combined_hulls/left_elbow_fe_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; visual mesh filename=./lsa1.1_new//meshes/urdf/obj_combined_hulls/left_elbow_fe_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
- link left_index_finger_dip_2_link: geometry collision mesh filename=./lsa1.1_new//meshes/urdf/obj_combined_hulls/left_index_fin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; visual mesh filename=./lsa1.1_new//meshes/urdf/obj_combined_hulls/left_index_fin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
- link left_index_finger_dip_link: geometry collision mesh filename=./lsa1.1_new//meshes/urdf/obj_combined_hulls/left_index_fin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; visual mesh filename=./lsa1.1_new//meshes/urdf/obj_combined_hulls/left_index_fin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
- link left_index_finger_mcp_abduction_link: geometry collision mesh filename=./lsa1.1_new//meshes/urdf/obj_combined_hulls/left_index_fin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; visual mesh filename=./lsa1.1_new//meshes/urdf/obj_combined_hulls/left_index_fin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
- link left_index_finger_mcp_flexion_2_link: geometry collision mesh filename=./lsa1.1_new//meshes/urdf/obj_combined_hulls/left_index_fin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; visual mesh filename=./lsa1.1_new//meshes/urdf/obj_combined_hulls/left_index_fin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
- link left_index_finger_mcp_flexion_link: geometry collision mesh filename=./lsa1.1_new//meshes/urdf/obj_combined_hulls/left_index_fin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; visual mesh filename=./lsa1.1_new//meshes/urdf/obj_combined_hulls/left_index_fin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
- link left_index_finger_pip_2_link: geometry collision mesh filename=./lsa1.1_new//meshes/urdf/obj_combined_hulls/left_index_fin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; visual mesh filename=./lsa1.1_new//meshes/urdf/obj_combined_hulls/left_index_fin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
- link left_index_finger_pip_link: geometry collision mesh filename=./lsa1.1_new//meshes/urdf/obj_combined_hulls/left_index_fin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; visual mesh filename=./lsa1.1_new//meshes/urdf/obj_combined_hulls/left_index_fin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
- link left_middle_finger_dip_2_link: geometry collision mesh filename=./lsa1.1_new//meshes/urdf/obj_combined_hulls/left_middle_fi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; visual mesh filename=./lsa1.1_new//meshes/urdf/obj_combined_hulls/left_middle_fi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
- link left_middle_finger_dip_link: geometry collision mesh filename=./lsa1.1_new//meshes/urdf/obj_combined_hulls/left_middle_fi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; visual mesh filename=./lsa1.1_new//meshes/urdf/obj_combined_hulls/left_middle_fi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
- link left_middle_finger_mcp_abduction_link: geometry collision mesh filename=./lsa1.1_new//meshes/urdf/obj_combined_hulls/left_middle_fi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; visual mesh filename=./lsa1.1_new//meshes/urdf/obj_combined_hulls/left_middle_fi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
- link left_middle_finger_mcp_flexion_2_link: geometry collision mesh filename=./lsa1.1_new//meshes/urdf/obj_combined_hulls/left_middle_fi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; visual mesh filename=./lsa1.1_new//meshes/urdf/obj_combined_hulls/left_middle_fi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
- link left_middle_finger_mcp_flexion_link: geometry collision mesh filename=./lsa1.1_new//meshes/urdf/obj_combined_hulls/left_middle_fi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; visual mesh filename=./lsa1.1_new//meshes/urdf/obj_combined_hulls/left_middle_fi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
- link left_middle_finger_pip_2_link: geometry collision mesh filename=./lsa1.1_new//meshes/urdf/obj_combined_hulls/left_middle_fi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; visual mesh filename=./lsa1.1_new//meshes/urdf/obj_combined_hulls/left_middle_fi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
- link left_middle_finger_pip_link: geometry collision mesh filename=./lsa1.1_new//meshes/urdf/obj_combined_hulls/left_middle_fi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; visual mesh filename=./lsa1.1_new//meshes/urdf/obj_combined_hulls/left_middle_fi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
- link left_pinkie_finger_dip_2_link: geometry collision mesh filename=./lsa1.1_new//meshes/urdf/obj_combined_hulls/left_pinkie_fi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; visual mesh filename=./lsa1.1_new//meshes/urdf/obj_combined_hulls/left_pinkie_fi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
- link left_pinkie_finger_dip_link: geometry collision mesh filename=./lsa1.1_new//meshes/urdf/obj_combined_hulls/left_pinkie_fi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; visual mesh filename=./lsa1.1_new//meshes/urdf/obj_combined_hulls/left_pinkie_fi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
- link left_pinkie_finger_mcp_abduction_link: geometry collision mesh filename=./lsa1.1_new//meshes/urdf/obj_combined_hulls/left_pinkie_fi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; visual mesh filename=./lsa1.1_new//meshes/urdf/obj_combined_hulls/left_pinkie_fi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
- link left_pinkie_finger_mcp_flexion_2_link: geometry collision mesh filename=./lsa1.1_new//meshes/urdf/obj_combined_hulls/left_pinkie_fi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; visual mesh filename=./lsa1.1_new//meshes/urdf/obj_combined_hulls/left_pinkie_fi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
- link left_pinkie_finger_mcp_flexion_link: geometry collision mesh filename=./lsa1.1_new//meshes/urdf/obj_combined_hulls/left_pinkie_fi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; visual mesh filename=./lsa1.1_new//meshes/urdf/obj_combined_hulls/left_pinkie_fi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
- link left_pinkie_finger_pip_2_link: geometry collision mesh filename=./lsa1.1_new//meshes/urdf/obj_combined_hulls/left_pinkie_fi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; visual mesh filename=./lsa1.1_new//meshes/urdf/obj_combined_hulls/left_pinkie_fi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
- link left_pinkie_finger_pip_link: geometry collision mesh filename=./lsa1.1_new//meshes/urdf/obj_combined_hulls/left_pinkie_fi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; visual mesh filename=./lsa1.1_new//meshes/urdf/obj_combined_hulls/left_pinkie_fi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
- link left_ring_finger_dip_2_link: geometry collision mesh filename=./lsa1.1_new//meshes/urdf/obj_combined_hulls/left_ring_fing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; visual mesh filename=./lsa1.1_new//meshes/urdf/obj_combined_hulls/left_ring_fing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
- link left_ring_finger_dip_link: geometry collision mesh filename=./lsa1.1_new//meshes/urdf/obj_combined_hulls/left_ring_fing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; visual mesh filename=./lsa1.1_new//meshes/urdf/obj_combined_hulls/left_ring_fing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
- link left_ring_finger_mcp_abduction_link: geometry collision mesh filename=./lsa1.1_new//meshes/urdf/obj_combined_hulls/left_ring_fing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; visual mesh filename=./lsa1.1_new//meshes/urdf/obj_combined_hulls/left_ring_fing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
- link left_ring_finger_mcp_flexion_2_link: geometry collision mesh filename=./lsa1.1_new//meshes/urdf/obj_combined_hulls/left_ring_fing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; visual mesh filename=./lsa1.1_new//meshes/urdf/obj_combined_hulls/left_ring_fing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
- link left_ring_finger_mcp_flexion_link: geometry collision mesh filename=./lsa1.1_new//meshes/urdf/obj_combined_hulls/left_ring_fing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; visual mesh filename=./lsa1.1_new//meshes/urdf/obj_combined_hulls/left_ring_fing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
- link left_ring_finger_pip_2_link: geometry collision mesh filename=./lsa1.1_new//meshes/urdf/obj_combined_hulls/left_ring_fing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; visual mesh filename=./lsa1.1_new//meshes/urdf/obj_combined_hulls/left_ring_fing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
- link left_ring_finger_pip_link: geometry collision mesh filename=./lsa1.1_new//meshes/urdf/obj_combined_hulls/left_ring_fing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; visual mesh filename=./lsa1.1_new//meshes/urdf/obj_combined_hulls/left_ring_fing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
- link left_shoulder_aa_link: geometry collision mesh filename=./lsa1.1_new//meshes/urdf/obj_combined_hulls/left_shoulder_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; visual mesh filename=./lsa1.1_new//meshes/urdf/obj_combined_hulls/left_shoulder_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
- link left_shoulder_fe_link: geometry collision mesh filename=./lsa1.1_new//meshes/urdf/obj_combined_hulls/left_shoulder_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; visual mesh filename=./lsa1.1_new//meshes/urdf/obj_combined_hulls/left_shoulder_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
- link left_shoulder_ie_link: geometry collision mesh filename=./lsa1.1_new//meshes/urdf/obj_combined_hulls/left_shoulder_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; visual mesh filename=./lsa1.1_new//meshes/urdf/obj_combined_hulls/left_shoulder_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
- link left_thumb_abduction_link: geometry collision mesh filename=./lsa1.1_new//meshes/urdf/obj_combined_hulls/left_thumb_abd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; visual mesh filename=./lsa1.1_new//meshes/urdf/obj_combined_hulls/left_thumb_abd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
- link left_thumb_dip_2_link: geometry collision mesh filename=./lsa1.1_new//meshes/urdf/obj_combined_hulls/left_thumb_dip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; visual mesh filename=./lsa1.1_new//meshes/urdf/obj_combined_hulls/left_thumb_dip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
- link left_thumb_dip_link: geometry collision mesh filename=./lsa1.1_new//meshes/urdf/obj_combined_hulls/left_thumb_dip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; visual mesh filename=./lsa1.1_new//meshes/urdf/obj_combined_hulls/left_thumb_dip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
- link left_thumb_mcp_flexion_2_link: geometry collision mesh filename=./lsa1.1_new//meshes/urdf/obj_combined_hulls/left_thumb_mcp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; visual mesh filename=./lsa1.1_new//meshes/urdf/obj_combined_hulls/left_thumb_mcp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
- link left_thumb_mcp_flexion_link: geometry collision mesh filename=./lsa1.1_new//meshes/urdf/obj_combined_hulls/left_thumb_mcp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; visual mesh filename=./lsa1.1_new//meshes/urdf/obj_combined_hulls/left_thumb_mcp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
- link left_thumb_opposition_2_link: geometry collision mesh filename=./lsa1.1_new//meshes/urdf/obj_combined_hulls/left_thumb_opp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; visual mesh filename=./lsa1.1_new//meshes/urdf/obj_combined_hulls/left_thumb_opp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
- link left_thumb_opposition_link: geometry collision mesh filename=./lsa1.1_new//meshes/urdf/obj_combined_hulls/left_thumb_opp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; visual mesh filename=./lsa1.1_new//meshes/urdf/obj_combined_hulls/left_thumb_opp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
- link left_wheel_link: geometry collision mesh filename=./lsa1.1_new//meshes/urdf/obj_combined_hulls/left_wheel_lin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; visual mesh filename=./lsa1.1_new//meshes/urdf/obj_combined_hulls/left_wheel_lin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
- link left_wrist_flexion_link: geometry collision mesh filename=./lsa1.1_new//meshes/urdf/obj_combined_hulls/left_wrist_fle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; visual mesh filename=./lsa1.1_new//meshes/urdf/obj_combined_hulls/left_wrist_fle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
- link left_wrist_rotation_link: geometry collision mesh filename=./lsa1.1_new//meshes/urdf/obj_combined_hulls/left_wrist_rot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; visual mesh filename=./lsa1.1_new//meshes/urdf/obj_combined_hulls/left_wrist_rot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
- link neck_pitch_link: geometry collision mesh filename=./lsa1.1_new//meshes/urdf/obj_combined_hulls/neck_pitch_lin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; visual mesh filename=./lsa1.1_new//meshes/urdf/obj_combined_hulls/neck_pitch_lin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
- link neck_roll_link: geometry collision mesh filename=./lsa1.1_new//meshes/urdf/obj_combined_hulls/neck_roll_link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; visual mesh filename=./lsa1.1_new//meshes/urdf/obj_combined_hulls/neck_roll_link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
- link neck_yaw_link: geometry collision mesh filename=./lsa1.1_new//meshes/urdf/obj_combined_hulls/neck_yaw_link.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; visual mesh filename=./lsa1.1_new//meshes/urdf/obj_combined_hulls/neck_yaw_link.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
- link right_caster_link: geometry collision mesh filename=./lsa1.1_new//meshes/urdf/obj_combined_hulls/right_caster_l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; visual mesh filename=./lsa1.1_new//meshes/urdf/obj_combined_hulls/right_caster_l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
- link right_caster_swivel_link: geometry collision mesh filename=./lsa1.1_new//meshes/urdf/obj_combined_hulls/right_caster_s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; visual mesh filename=./lsa1.1_new//meshes/urdf/obj_combined_hulls/right_caster_s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
- link right_elbow_fe_link: geometry collision mesh filename=./lsa1.1_new//meshes/urdf/obj_combined_hulls/right_elbow_fe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; visual mesh filename=./lsa1.1_new//meshes/urdf/obj_combined_hulls/right_elbow_fe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
- link right_index_finger_dip_2_link: geometry collision mesh filename=./lsa1.1_new//meshes/urdf/obj_combined_hulls/right_index_fi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; visual mesh filename=./lsa1.1_new//meshes/urdf/obj_combined_hulls/right_index_fi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
- link right_index_finger_dip_link: geometry collision mesh filename=./lsa1.1_new//meshes/urdf/obj_combined_hulls/right_index_fi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; visual mesh filename=./lsa1.1_new//meshes/urdf/obj_combined_hulls/right_index_fi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
- link right_index_finger_mcp_abduction_link: geometry collision mesh filename=./lsa1.1_new//meshes/urdf/obj_combined_hulls/right_index_fi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; visual mesh filename=./lsa1.1_new//meshes/urdf/obj_combined_hulls/right_index_fi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
- link right_index_finger_mcp_flexion_2_link: geometry collision mesh filename=./lsa1.1_new//meshes/urdf/obj_combined_hulls/right_index_fi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; visual mesh filename=./lsa1.1_new//meshes/urdf/obj_combined_hulls/right_index_fi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
- link right_index_finger_mcp_flexion_link: geometry collision mesh filename=./lsa1.1_new//meshes/urdf/obj_combined_hulls/right_index_fi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; visual mesh filename=./lsa1.1_new//meshes/urdf/obj_combined_hulls/right_index_fi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
- link right_index_finger_pip_2_link: geometry collision mesh filename=./lsa1.1_new//meshes/urdf/obj_combined_hulls/right_index_fi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; visual mesh filename=./lsa1.1_new//meshes/urdf/obj_combined_hulls/right_index_fi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
- link right_index_finger_pip_link: geometry collision mesh filename=./lsa1.1_new//meshes/urdf/obj_combined_hulls/right_index_fi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; visual mesh filename=./lsa1.1_new//meshes/urdf/obj_combined_hulls/right_index_fi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
- link right_middle_finger_dip_2_link: geometry collision mesh filename=./lsa1.1_new//meshes/urdf/obj_combined_hulls/right_middle_f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; visual mesh filename=./lsa1.1_new//meshes/urdf/obj_combined_hulls/right_middle_f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
- link right_middle_finger_dip_link: geometry collision mesh filename=./lsa1.1_new//meshes/urdf/obj_combined_hulls/right_middle_f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; visual mesh filename=./lsa1.1_new//meshes/urdf/obj_combined_hulls/right_middle_f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
- link right_middle_finger_mcp_abduction_link: geometry collision mesh filename=./lsa1.1_new//meshes/urdf/obj_combined_hulls/right_middle_f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; visual mesh filename=./lsa1.1_new//meshes/urdf/obj_combined_hulls/right_middle_f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
- link right_middle_finger_mcp_flexion_2_link: geometry collision mesh filename=./lsa1.1_new//meshes/urdf/obj_combined_hulls/right_middle_f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; visual mesh filename=./lsa1.1_new//meshes/urdf/obj_combined_hulls/right_middle_f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
- link right_middle_finger_mcp_flexion_link: geometry collision mesh filename=./lsa1.1_new//meshes/urdf/obj_combined_hulls/right_middle_f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; visual mesh filename=./lsa1.1_new//meshes/urdf/obj_combined_hulls/right_middle_f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
- link right_middle_finger_pip_2_link: geometry collision mesh filename=./lsa1.1_new//meshes/urdf/obj_combined_hulls/right_middle_f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; visual mesh filename=./lsa1.1_new//meshes/urdf/obj_combined_hulls/right_middle_f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
- link right_middle_finger_pip_link: geometry collision mesh filename=./lsa1.1_new//meshes/urdf/obj_combined_hulls/right_middle_f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; visual mesh filename=./lsa1.1_new//meshes/urdf/obj_combined_hulls/right_middle_f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
- link right_pinkie_finger_dip_2_link: geometry collision mesh filename=./lsa1.1_new//meshes/urdf/obj_combined_hulls/right_pinkie_f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; visual mesh filename=./lsa1.1_new//meshes/urdf/obj_combined_hulls/right_pinkie_f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
- link right_pinkie_finger_dip_link: geometry collision mesh filename=./lsa1.1_new//meshes/urdf/obj_combined_hulls/right_pinkie_f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; visual mesh filename=./lsa1.1_new//meshes/urdf/obj_combined_hulls/right_pinkie_f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
- link right_pinkie_finger_mcp_abduction_link: geometry collision mesh filename=./lsa1.1_new//meshes/urdf/obj_combined_hulls/right_pinkie_f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; visual mesh filename=./lsa1.1_new//meshes/urdf/obj_combined_hulls/right_pinkie_f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
- link right_pinkie_finger_mcp_flexion_2_link: geometry collision mesh filename=./lsa1.1_new//meshes/urdf/obj_combined_hulls/right_pinkie_f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; visual mesh filename=./lsa1.1_new//meshes/urdf/obj_combined_hulls/right_pinkie_f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
- link right_pinkie_finger_mcp_flexion_link: geometry collision mesh filename=./lsa1.1_new//meshes/urdf/obj_combined_hulls/right_pinkie_f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; visual mesh filename=./lsa1.1_new//meshes/urdf/obj_combined_hulls/right_pinkie_f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
- link right_pinkie_finger_pip_2_link: geometry collision mesh filename=./lsa1.1_new//meshes/urdf/obj_combined_hulls/right_pinkie_f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; visual mesh filename=./lsa1.1_new//meshes/urdf/obj_combined_hulls/right_pinkie_f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
- link right_pinkie_finger_pip_link: geometry collision mesh filename=./lsa1.1_new//meshes/urdf/obj_combined_hulls/right_pinkie_f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; visual mesh filename=./lsa1.1_new//meshes/urdf/obj_combined_hulls/right_pinkie_f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
- link right_ring_finger_dip_2_link: geometry collision mesh filename=./lsa1.1_new//meshes/urdf/obj_combined_hulls/right_ring_fin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; visual mesh filename=./lsa1.1_new//meshes/urdf/obj_combined_hulls/right_ring_fin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
- link right_ring_finger_dip_link: geometry collision mesh filename=./lsa1.1_new//meshes/urdf/obj_combined_hulls/right_ring_fin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; visual mesh filename=./lsa1.1_new//meshes/urdf/obj_combined_hulls/right_ring_fin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
- link right_ring_finger_mcp_abduction_link: geometry collision mesh filename=./lsa1.1_new//meshes/urdf/obj_combined_hulls/right_ring_fin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; visual mesh filename=./lsa1.1_new//meshes/urdf/obj_combined_hulls/right_ring_fin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
- link right_ring_finger_mcp_flexion_2_link: geometry collision mesh filename=./lsa1.1_new//meshes/urdf/obj_combined_hulls/right_ring_fin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; visual mesh filename=./lsa1.1_new//meshes/urdf/obj_combined_hulls/right_ring_fin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
- link right_ring_finger_mcp_flexion_link: geometry collision mesh filename=./lsa1.1_new//meshes/urdf/obj_combined_hulls/right_ring_fin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; visual mesh filename=./lsa1.1_new//meshes/urdf/obj_combined_hulls/right_ring_fin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
- link right_ring_finger_pip_2_link: geometry collision mesh filename=./lsa1.1_new//meshes/urdf/obj_combined_hulls/right_ring_fin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; visual mesh filename=./lsa1.1_new//meshes/urdf/obj_combined_hulls/right_ring_fin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
- link right_ring_finger_pip_link: geometry collision mesh filename=./lsa1.1_new//meshes/urdf/obj_combined_hulls/right_ring_fin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; visual mesh filename=./lsa1.1_new//meshes/urdf/obj_combined_hulls/right_ring_fin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
- link right_shoulder_aa_link: geometry collision mesh filename=./lsa1.1_new//meshes/urdf/obj_combined_hulls/right_shoulder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; visual mesh filename=./lsa1.1_new//meshes/urdf/obj_combined_hulls/right_shoulder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
- link right_shoulder_fe_link: geometry collision mesh filename=./lsa1.1_new//meshes/urdf/obj_combined_hulls/right_shoulder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; visual mesh filename=./lsa1.1_new//meshes/urdf/obj_combined_hulls/right_shoulder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
- link right_shoulder_ie_link: geometry collision mesh filename=./lsa1.1_new//meshes/urdf/obj_combined_hulls/right_shoulder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; visual mesh filename=./lsa1.1_new//meshes/urdf/obj_combined_hulls/right_shoulder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
- link right_thumb_abduction_link: geometry collision mesh filename=./lsa1.1_new//meshes/urdf/obj_combined_hulls/right_thumb_ab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; visual mesh filename=./lsa1.1_new//meshes/urdf/obj_combined_hulls/right_thumb_ab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
- link right_thumb_dip_2_link: geometry collision mesh filename=./lsa1.1_new//meshes/urdf/obj_combined_hulls/right_thumb_di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; visual mesh filename=./lsa1.1_new//meshes/urdf/obj_combined_hulls/right_thumb_di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
- link right_thumb_dip_link: geometry collision mesh filename=./lsa1.1_new//meshes/urdf/obj_combined_hulls/right_thumb_di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; visual mesh filename=./lsa1.1_new//meshes/urdf/obj_combined_hulls/right_thumb_di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
- link right_thumb_mcp_flexion_2_link: geometry collision mesh filename=./lsa1.1_new//meshes/urdf/obj_combined_hulls/right_thumb_mc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; visual mesh filename=./lsa1.1_new//meshes/urdf/obj_combined_hulls/right_thumb_mc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
- link right_thumb_mcp_flexion_link: geometry collision mesh filename=./lsa1.1_new//meshes/urdf/obj_combined_hulls/right_thumb_mc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; visual mesh filename=./lsa1.1_new//meshes/urdf/obj_combined_hulls/right_thumb_mc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
- link right_thumb_opposition_2_link: geometry collision mesh filename=./lsa1.1_new//meshes/urdf/obj_combined_hulls/right_thumb_op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; visual mesh filename=./lsa1.1_new//meshes/urdf/obj_combined_hulls/right_thumb_op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
- link right_thumb_opposition_link: geometry collision mesh filename=./lsa1.1_new//meshes/urdf/obj_combined_hulls/right_thumb_op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; visual mesh filename=./lsa1.1_new//meshes/urdf/obj_combined_hulls/right_thumb_op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
- link right_wheel_link: geometry collision mesh filename=./lsa1.1_new//meshes/urdf/obj_combined_hulls/right_wheel_li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; visual mesh filename=./lsa1.1_new//meshes/urdf/obj_combined_hulls/right_wheel_li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
- link right_wrist_flexion_link: geometry collision mesh filename=./lsa1.1_new//meshes/urdf/obj_combined_hulls/right_wrist_fl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; visual mesh filename=./lsa1.1_new//meshes/urdf/obj_combined_hulls/right_wrist_fl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
- link right_wrist_rotation_link: geometry collision mesh filename=./lsa1.1_new//meshes/urdf/obj_combined_hulls/right_wrist_ro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; visual mesh filename=./lsa1.1_new//meshes/urdf/obj_combined_hulls/right_wrist_ro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
- link root_link: geometry collision mesh filename=./lsa1.1_new//meshes/urdf/obj_combined_hulls/root_link.obj; visual mesh filename=./lsa1.1_new//meshes/urdf/obj_combined_hulls/root_link.obj
- link torso_pitch_lower_link: geometry collision mesh filename=./lsa1.1_new//meshes/urdf/obj_combined_hulls/torso_pitch_lo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; visual mesh filename=./lsa1.1_new//meshes/urdf/obj_combined_hulls/torso_pitch_lo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
- link torso_pitch_upper_link: geometry collision mesh filename=./lsa1.1_new//meshes/urdf/obj_combined_hulls/torso_pitch_up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; visual mesh filename=./lsa1.1_new//meshes/urdf/obj_combined_hulls/torso_pitch_up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
- link torso_yaw_link: geometry collision mesh filename=./lsa1.1_new//meshes/urdf/obj_combined_hulls/torso_yaw_link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; visual mesh filename=./lsa1.1_new//meshes/urdf/obj_combined_hulls/torso_yaw_link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
