Commit message: one more change to file location in robot_obj_combined_hulls.urdf

File: lsa1.1_new/robot_obj_combined_hulls.urdf (robot description, URDF)
Before this commit: robot LSA, 146 links, 145 joints
Links:
- link column_link: geometry collision mesh filename=.//meshes/urdf/obj_combined_hulls/column_link.obj; visual mesh filename=.//meshes/urdf/obj_combined_hulls/column_link.obj
- link hydraulic_container_link: geometry collision mesh filename=.//meshes/urdf/obj_combined_hulls/hydraulic_container_link.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; visual mesh filename=.//meshes/urdf/obj_combined_hulls/hydraulic_container_link.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
- link left_caster_link: geometry collision mesh filename=.//meshes/urdf/obj_combined_hulls/left_caster_link.obj; visual mesh filename=.//meshes/urdf/obj_combined_hulls/left_caster_link.obj
- link left_caster_swivel_link: geometry collision mesh filename=.//meshes/urdf/obj_combined_hulls/left_caster_swivel_link.o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; visual mesh filename=.//meshes/urdf/obj_combined_hulls/left_caster_swivel_link.o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
- link left_elbow_fe_link: geometry collision mesh filename=.//meshes/urdf/obj_combined_hulls/left_elbow_fe_link.obj; visual mesh filename=.//meshes/urdf/obj_combined_hulls/left_elbow_fe_link.obj
- link left_index_finger_dip_2_link: geometry collision mesh filename=.//meshes/urdf/obj_combined_hulls/left_index_finger_dip_2_l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; visual mesh filename=.//meshes/urdf/obj_combined_hulls/left_index_finger_dip_2_l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
- link left_index_finger_dip_link: geometry collision mesh filename=.//meshes/urdf/obj_combined_hulls/left_index_finger_dip_lin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; visual mesh filename=.//meshes/urdf/obj_combined_hulls/left_index_finger_dip_lin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
- link left_index_finger_mcp_abduction_link: geometry collision mesh filename=.//meshes/urdf/obj_combined_hulls/left_index_finger_mcp_abd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; visual mesh filename=.//meshes/urdf/obj_combined_hulls/left_index_finger_mcp_abd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
- link left_index_finger_mcp_flexion_2_link: geometry collision mesh filename=.//meshes/urdf/obj_combined_hulls/left_index_finger_mcp_fle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; visual mesh filename=.//meshes/urdf/obj_combined_hulls/left_index_finger_mcp_fle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
- link left_index_finger_mcp_flexion_link: geometry collision mesh filename=.//meshes/urdf/obj_combined_hulls/left_index_finger_mcp_fle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; visual mesh filename=.//meshes/urdf/obj_combined_hulls/left_index_finger_mcp_fle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
- link left_index_finger_pip_2_link: geometry collision mesh filename=.//meshes/urdf/obj_combined_hulls/left_index_finger_pip_2_l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; visual mesh filename=.//meshes/urdf/obj_combined_hulls/left_index_finger_pip_2_l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
- link left_index_finger_pip_link: geometry collision mesh filename=.//meshes/urdf/obj_combined_hulls/left_index_finger_pip_lin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; visual mesh filename=.//meshes/urdf/obj_combined_hulls/left_index_finger_pip_lin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
- link left_middle_finger_dip_2_link: geometry collision mesh filename=.//meshes/urdf/obj_combined_hulls/left_middle_finger_dip_2_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; visual mesh filename=.//meshes/urdf/obj_combined_hulls/left_middle_finger_dip_2_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
- link left_middle_finger_dip_link: geometry collision mesh filename=.//meshes/urdf/obj_combined_hulls/left_middle_finger_dip_li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; visual mesh filename=.//meshes/urdf/obj_combined_hulls/left_middle_finger_dip_li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
- link left_middle_finger_mcp_abduction_link: geometry collision mesh filename=.//meshes/urdf/obj_combined_hulls/left_middle_finger_mcp_ab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; visual mesh filename=.//meshes/urdf/obj_combined_hulls/left_middle_finger_mcp_ab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
- link left_middle_finger_mcp_flexion_2_link: geometry collision mesh filename=.//meshes/urdf/obj_combined_hulls/left_middle_finger_mcp_fl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; visual mesh filename=.//meshes/urdf/obj_combined_hulls/left_middle_finger_mcp_fl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
- link left_middle_finger_mcp_flexion_link: geometry collision mesh filename=.//meshes/urdf/obj_combined_hulls/left_middle_finger_mcp_fl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; visual mesh filename=.//meshes/urdf/obj_combined_hulls/left_middle_finger_mcp_fl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
- link left_middle_finger_pip_2_link: geometry collision mesh filename=.//meshes/urdf/obj_combined_hulls/left_middle_finger_pip_2_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; visual mesh filename=.//meshes/urdf/obj_combined_hulls/left_middle_finger_pip_2_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
- link left_middle_finger_pip_link: geometry collision mesh filename=.//meshes/urdf/obj_combined_hulls/left_middle_finger_pip_li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; visual mesh filename=.//meshes/urdf/obj_combined_hulls/left_middle_finger_pip_li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
- link left_pinkie_finger_dip_2_link: geometry collision mesh filename=.//meshes/urdf/obj_combined_hulls/left_pinkie_finger_dip_2_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; visual mesh filename=.//meshes/urdf/obj_combined_hulls/left_pinkie_finger_dip_2_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
- link left_pinkie_finger_dip_link: geometry collision mesh filename=.//meshes/urdf/obj_combined_hulls/left_pinkie_finger_dip_li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; visual mesh filename=.//meshes/urdf/obj_combined_hulls/left_pinkie_finger_dip_li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
- link left_pinkie_finger_mcp_abduction_link: geometry collision mesh filename=.//meshes/urdf/obj_combined_hulls/left_pinkie_finger_mcp_ab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; visual mesh filename=.//meshes/urdf/obj_combined_hulls/left_pinkie_finger_mcp_ab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
- link left_pinkie_finger_mcp_flexion_2_link: geometry collision mesh filename=.//meshes/urdf/obj_combined_hulls/left_pinkie_finger_mcp_fl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; visual mesh filename=.//meshes/urdf/obj_combined_hulls/left_pinkie_finger_mcp_fl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
- link left_pinkie_finger_mcp_flexion_link: geometry collision mesh filename=.//meshes/urdf/obj_combined_hulls/left_pinkie_finger_mcp_fl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; visual mesh filename=.//meshes/urdf/obj_combined_hulls/left_pinkie_finger_mcp_fl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
- link left_pinkie_finger_pip_2_link: geometry collision mesh filename=.//meshes/urdf/obj_combined_hulls/left_pinkie_finger_pip_2_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; visual mesh filename=.//meshes/urdf/obj_combined_hulls/left_pinkie_finger_pip_2_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
- link left_pinkie_finger_pip_link: geometry collision mesh filename=.//meshes/urdf/obj_combined_hulls/left_pinkie_finger_pip_li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; visual mesh filename=.//meshes/urdf/obj_combined_hulls/left_pinkie_finger_pip_li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
- link left_ring_finger_dip_2_link: geometry collision mesh filename=.//meshes/urdf/obj_combined_hulls/left_ring_finger_dip_2_li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; visual mesh filename=.//meshes/urdf/obj_combined_hulls/left_ring_finger_dip_2_li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
- link left_ring_finger_dip_link: geometry collision mesh filename=.//meshes/urdf/obj_combined_hulls/left_ring_finger_dip_link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; visual mesh filename=.//meshes/urdf/obj_combined_hulls/left_ring_finger_dip_link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
- link left_ring_finger_mcp_abduction_link: geometry collision mesh filename=.//meshes/urdf/obj_combined_hulls/left_ring_finger_mcp_abdu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; visual mesh filename=.//meshes/urdf/obj_combined_hulls/left_ring_finger_mcp_abdu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
- link left_ring_finger_mcp_flexion_2_link: geometry collision mesh filename=.//meshes/urdf/obj_combined_hulls/left_ring_finger_mcp_flex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; visual mesh filename=.//meshes/urdf/obj_combined_hulls/left_ring_finger_mcp_flex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
- link left_ring_finger_mcp_flexion_link: geometry collision mesh filename=.//meshes/urdf/obj_combined_hulls/left_ring_finger_mcp_flex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; visual mesh filename=.//meshes/urdf/obj_combined_hulls/left_ring_finger_mcp_flex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
- link left_ring_finger_pip_2_link: geometry collision mesh filename=.//meshes/urdf/obj_combined_hulls/left_ring_finger_pip_2_li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; visual mesh filename=.//meshes/urdf/obj_combined_hulls/left_ring_finger_pip_2_li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
- link left_ring_finger_pip_link: geometry collision mesh filename=.//meshes/urdf/obj_combined_hulls/left_ring_finger_pip_link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; visual mesh filename=.//meshes/urdf/obj_combined_hulls/left_ring_finger_pip_link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
- link left_shoulder_aa_link: geometry collision mesh filename=.//meshes/urdf/obj_combined_hulls/left_shoulder_aa_link.obj; visual mesh filename=.//meshes/urdf/obj_combined_hulls/left_shoulder_aa_link.obj
- link left_shoulder_fe_link: geometry collision mesh filename=.//meshes/urdf/obj_combined_hulls/left_shoulder_fe_link.obj; visual mesh filename=.//meshes/urdf/obj_combined_hulls/left_shoulder_fe_link.obj
- link left_shoulder_ie_link: geometry collision mesh filename=.//meshes/urdf/obj_combined_hulls/left_shoulder_ie_link.obj; visual mesh filename=.//meshes/urdf/obj_combined_hulls/left_shoulder_ie_link.obj
- link left_thumb_abduction_link: geometry collision mesh filename=.//meshes/urdf/obj_combined_hulls/left_thumb_abduction_link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; visual mesh filename=.//meshes/urdf/obj_combined_hulls/left_thumb_abduction_link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
- link left_thumb_dip_2_link: geometry collision mesh filename=.//meshes/urdf/obj_combined_hulls/left_thumb_dip_2_link.obj; visual mesh filename=.//meshes/urdf/obj_combined_hulls/left_thumb_dip_2_link.obj
- link left_thumb_dip_link: geometry collision mesh filename=.//meshes/urdf/obj_combined_hulls/left_thumb_dip_link.obj; visual mesh filename=.//meshes/urdf/obj_combined_hulls/left_thumb_dip_link.obj
- link left_thumb_mcp_flexion_2_link: geometry collision mesh filename=.//meshes/urdf/obj_combined_hulls/left_thumb_mcp_flexion_2_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; visual mesh filename=.//meshes/urdf/obj_combined_hulls/left_thumb_mcp_flexion_2_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
- link left_thumb_mcp_flexion_link: geometry collision mesh filename=.//meshes/urdf/obj_combined_hulls/left_thumb_mcp_flexion_li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; visual mesh filename=.//meshes/urdf/obj_combined_hulls/left_thumb_mcp_flexion_li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
- link left_thumb_opposition_2_link: geometry collision mesh filename=.//meshes/urdf/obj_combined_hulls/left_thumb_opposition_2_l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; visual mesh filename=.//meshes/urdf/obj_combined_hulls/left_thumb_opposition_2_l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
- link left_thumb_opposition_link: geometry collision mesh filename=.//meshes/urdf/obj_combined_hulls/left_thumb_opposition_lin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; visual mesh filename=.//meshes/urdf/obj_combined_hulls/left_thumb_opposition_lin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
- link left_wheel_link: geometry collision mesh filename=.//meshes/urdf/obj_combined_hulls/left_wheel_link.obj; visual mesh filename=.//meshes/urdf/obj_combined_hulls/left_wheel_link.obj
- link left_wrist_flexion_link: geometry collision mesh filename=.//meshes/urdf/obj_combined_hulls/left_wrist_flexion_link.o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; visual mesh filename=.//meshes/urdf/obj_combined_hulls/left_wrist_flexion_link.o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
- link left_wrist_rotation_link: geometry collision mesh filename=.//meshes/urdf/obj_combined_hulls/left_wrist_rotation_link.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; visual mesh filename=.//meshes/urdf/obj_combined_hulls/left_wrist_rotation_link.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
- link neck_pitch_link: geometry collision mesh filename=.//meshes/urdf/obj_combined_hulls/neck_pitch_link.obj; visual mesh filename=.//meshes/urdf/obj_combined_hulls/neck_pitch_link.obj
- link neck_roll_link: geometry collision mesh filename=.//meshes/urdf/obj_combined_hulls/neck_roll_link.obj; visual mesh filename=.//meshes/urdf/obj_combined_hulls/neck_roll_link.obj
- link neck_yaw_link: geometry collision mesh filename=.//meshes/urdf/obj_combined_hulls/neck_yaw_link.obj; visual mesh filename=.//meshes/urdf/obj_combined_hulls/neck_yaw_link.obj
- link right_caster_link: geometry collision mesh filename=.//meshes/urdf/obj_combined_hulls/right_caster_link.obj; visual mesh filename=.//meshes/urdf/obj_combined_hulls/right_caster_link.obj
- link right_caster_swivel_link: geometry collision mesh filename=.//meshes/urdf/obj_combined_hulls/right_caster_swivel_link.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; visual mesh filename=.//meshes/urdf/obj_combined_hulls/right_caster_swivel_link.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
- link right_elbow_fe_link: geometry collision mesh filename=.//meshes/urdf/obj_combined_hulls/right_elbow_fe_link.obj; visual mesh filename=.//meshes/urdf/obj_combined_hulls/right_elbow_fe_link.obj
- link right_index_finger_dip_2_link: geometry collision mesh filename=.//meshes/urdf/obj_combined_hulls/right_index_finger_dip_2_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; visual mesh filename=.//meshes/urdf/obj_combined_hulls/right_index_finger_dip_2_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
- link right_index_finger_dip_link: geometry collision mesh filename=.//meshes/urdf/obj_combined_hulls/right_index_finger_dip_li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; visual mesh filename=.//meshes/urdf/obj_combined_hulls/right_index_finger_dip_li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
- link right_index_finger_mcp_abduction_link: geometry collision mesh filename=.//meshes/urdf/obj_combined_hulls/right_index_finger_mcp_ab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; visual mesh filename=.//meshes/urdf/obj_combined_hulls/right_index_finger_mcp_ab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
- link right_index_finger_mcp_flexion_2_link: geometry collision mesh filename=.//meshes/urdf/obj_combined_hulls/right_index_finger_mcp_fl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; visual mesh filename=.//meshes/urdf/obj_combined_hulls/right_index_finger_mcp_fl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
- link right_index_finger_mcp_flexion_link: geometry collision mesh filename=.//meshes/urdf/obj_combined_hulls/right_index_finger_mcp_fl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; visual mesh filename=.//meshes/urdf/obj_combined_hulls/right_index_finger_mcp_fl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
- link right_index_finger_pip_2_link: geometry collision mesh filename=.//meshes/urdf/obj_combined_hulls/right_index_finger_pip_2_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; visual mesh filename=.//meshes/urdf/obj_combined_hulls/right_index_finger_pip_2_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
- link right_index_finger_pip_link: geometry collision mesh filename=.//meshes/urdf/obj_combined_hulls/right_index_finger_pip_li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; visual mesh filename=.//meshes/urdf/obj_combined_hulls/right_index_finger_pip_li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
- link right_middle_finger_dip_2_link: geometry collision mesh filename=.//meshes/urdf/obj_combined_hulls/right_middle_finger_dip_2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; visual mesh filename=.//meshes/urdf/obj_combined_hulls/right_middle_finger_dip_2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
- link right_middle_finger_dip_link: geometry collision mesh filename=.//meshes/urdf/obj_combined_hulls/right_middle_finger_dip_l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; visual mesh filename=.//meshes/urdf/obj_combined_hulls/right_middle_finger_dip_l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
- link right_middle_finger_mcp_abduction_link: geometry collision mesh filename=.//meshes/urdf/obj_combined_hulls/right_middle_finger_mcp_a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; visual mesh filename=.//meshes/urdf/obj_combined_hulls/right_middle_finger_mcp_a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
- link right_middle_finger_mcp_flexion_2_link: geometry collision mesh filename=.//meshes/urdf/obj_combined_hulls/right_middle_finger_mcp_f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; visual mesh filename=.//meshes/urdf/obj_combined_hulls/right_middle_finger_mcp_f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
- link right_middle_finger_mcp_flexion_link: geometry collision mesh filename=.//meshes/urdf/obj_combined_hulls/right_middle_finger_mcp_f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; visual mesh filename=.//meshes/urdf/obj_combined_hulls/right_middle_finger_mcp_f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
- link right_middle_finger_pip_2_link: geometry collision mesh filename=.//meshes/urdf/obj_combined_hulls/right_middle_finger_pip_2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; visual mesh filename=.//meshes/urdf/obj_combined_hulls/right_middle_finger_pip_2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
- link right_middle_finger_pip_link: geometry collision mesh filename=.//meshes/urdf/obj_combined_hulls/right_middle_finger_pip_l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; visual mesh filename=.//meshes/urdf/obj_combined_hulls/right_middle_finger_pip_l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
- link right_pinkie_finger_dip_2_link: geometry collision mesh filename=.//meshes/urdf/obj_combined_hulls/right_pinkie_finger_dip_2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; visual mesh filename=.//meshes/urdf/obj_combined_hulls/right_pinkie_finger_dip_2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
- link right_pinkie_finger_dip_link: geometry collision mesh filename=.//meshes/urdf/obj_combined_hulls/right_pinkie_finger_dip_l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; visual mesh filename=.//meshes/urdf/obj_combined_hulls/right_pinkie_finger_dip_l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
- link right_pinkie_finger_mcp_abduction_link: geometry collision mesh filename=.//meshes/urdf/obj_combined_hulls/right_pinkie_finger_mcp_a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; visual mesh filename=.//meshes/urdf/obj_combined_hulls/right_pinkie_finger_mcp_a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
- link right_pinkie_finger_mcp_flexion_2_link: geometry collision mesh filename=.//meshes/urdf/obj_combined_hulls/right_pinkie_finger_mcp_f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; visual mesh filename=.//meshes/urdf/obj_combined_hulls/right_pinkie_finger_mcp_f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
- link right_pinkie_finger_mcp_flexion_link: geometry collision mesh filename=.//meshes/urdf/obj_combined_hulls/right_pinkie_finger_mcp_f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; visual mesh filename=.//meshes/urdf/obj_combined_hulls/right_pinkie_finger_mcp_f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
- link right_pinkie_finger_pip_2_link: geometry collision mesh filename=.//meshes/urdf/obj_combined_hulls/right_pinkie_finger_pip_2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; visual mesh filename=.//meshes/urdf/obj_combined_hulls/right_pinkie_finger_pip_2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
- link right_pinkie_finger_pip_link: geometry collision mesh filename=.//meshes/urdf/obj_combined_hulls/right_pinkie_finger_pip_l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; visual mesh filename=.//meshes/urdf/obj_combined_hulls/right_pinkie_finger_pip_l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
- link right_ring_finger_dip_2_link: geometry collision mesh filename=.//meshes/urdf/obj_combined_hulls/right_ring_finger_dip_2_l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; visual mesh filename=.//meshes/urdf/obj_combined_hulls/right_ring_finger_dip_2_l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
- link right_ring_finger_dip_link: geometry collision mesh filename=.//meshes/urdf/obj_combined_hulls/right_ring_finger_dip_lin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; visual mesh filename=.//meshes/urdf/obj_combined_hulls/right_ring_finger_dip_lin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
- link right_ring_finger_mcp_abduction_link: geometry collision mesh filename=.//meshes/urdf/obj_combined_hulls/right_ring_finger_mcp_abd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; visual mesh filename=.//meshes/urdf/obj_combined_hulls/right_ring_finger_mcp_abd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
- link right_ring_finger_mcp_flexion_2_link: geometry collision mesh filename=.//meshes/urdf/obj_combined_hulls/right_ring_finger_mcp_fle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; visual mesh filename=.//meshes/urdf/obj_combined_hulls/right_ring_finger_mcp_fle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
- link right_ring_finger_mcp_flexion_link: geometry collision mesh filename=.//meshes/urdf/obj_combined_hulls/right_ring_finger_mcp_fle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; visual mesh filename=.//meshes/urdf/obj_combined_hulls/right_ring_finger_mcp_fle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
- link right_ring_finger_pip_2_link: geometry collision mesh filename=.//meshes/urdf/obj_combined_hulls/right_ring_finger_pip_2_l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; visual mesh filename=.//meshes/urdf/obj_combined_hulls/right_ring_finger_pip_2_l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
- link right_ring_finger_pip_link: geometry collision mesh filename=.//meshes/urdf/obj_combined_hulls/right_ring_finger_pip_lin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; visual mesh filename=.//meshes/urdf/obj_combined_hulls/right_ring_finger_pip_lin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
- link right_shoulder_aa_link: geometry collision mesh filename=.//meshes/urdf/obj_combined_hulls/right_shoulder_aa_link.obj; visual mesh filename=.//meshes/urdf/obj_combined_hulls/right_shoulder_aa_link.obj
- link right_shoulder_fe_link: geometry collision mesh filename=.//meshes/urdf/obj_combined_hulls/right_shoulder_fe_link.obj; visual mesh filename=.//meshes/urdf/obj_combined_hulls/right_shoulder_fe_link.obj
- link right_shoulder_ie_link: geometry collision mesh filename=.//meshes/urdf/obj_combined_hulls/right_shoulder_ie_link.obj; visual mesh filename=.//meshes/urdf/obj_combined_hulls/right_shoulder_ie_link.obj
- link right_thumb_abduction_link: geometry collision mesh filename=.//meshes/urdf/obj_combined_hulls/right_thumb_abduction_lin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; visual mesh filename=.//meshes/urdf/obj_combined_hulls/right_thumb_abduction_lin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
- link right_thumb_dip_2_link: geometry collision mesh filename=.//meshes/urdf/obj_combined_hulls/right_thumb_dip_2_link.obj; visual mesh filename=.//meshes/urdf/obj_combined_hulls/right_thumb_dip_2_link.obj
- link right_thumb_dip_link: geometry collision mesh filename=.//meshes/urdf/obj_combined_hulls/right_thumb_dip_link.obj; visual mesh filename=.//meshes/urdf/obj_combined_hulls/right_thumb_dip_link.obj
- link right_thumb_mcp_flexion_2_link: geometry collision mesh filename=.//meshes/urdf/obj_combined_hulls/right_thumb_mcp_flexion_2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; visual mesh filename=.//meshes/urdf/obj_combined_hulls/right_thumb_mcp_flexion_2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
- link right_thumb_mcp_flexion_link: geometry collision mesh filename=.//meshes/urdf/obj_combined_hulls/right_thumb_mcp_flexion_l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; visual mesh filename=.//meshes/urdf/obj_combined_hulls/right_thumb_mcp_flexion_l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
- link right_thumb_opposition_2_link: geometry collision mesh filename=.//meshes/urdf/obj_combined_hulls/right_thumb_opposition_2_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; visual mesh filename=.//meshes/urdf/obj_combined_hulls/right_thumb_opposition_2_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
- link right_thumb_opposition_link: geometry collision mesh filename=.//meshes/urdf/obj_combined_hulls/right_thumb_opposition_li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; visual mesh filename=.//meshes/urdf/obj_combined_hulls/right_thumb_opposition_li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
- link right_wheel_link: geometry collision mesh filename=.//meshes/urdf/obj_combined_hulls/right_wheel_link.obj; visual mesh filename=.//meshes/urdf/obj_combined_hulls/right_wheel_link.obj
- link right_wrist_flexion_link: geometry collision mesh filename=.//meshes/urdf/obj_combined_hulls/right_wrist_flexion_link.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; visual mesh filename=.//meshes/urdf/obj_combined_hulls/right_wrist_flexion_link.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
- link right_wrist_rotation_link: geometry collision mesh filename=.//meshes/urdf/obj_combined_hulls/right_wrist_rotation_link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; visual mesh filename=.//meshes/urdf/obj_combined_hulls/right_wrist_rotation_link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
- link root_link: geometry collision mesh filename=.//meshes/urdf/obj_combined_hulls/root_link.obj; visual mesh filename=.//meshes/urdf/obj_combined_hulls/root_link.obj
- link torso_pitch_lower_link: geometry collision mesh filename=.//meshes/urdf/obj_combined_hulls/torso_pitch_lower_link.obj; visual mesh filename=.//meshes/urdf/obj_combined_hulls/torso_pitch_lower_link.obj
- link torso_pitch_upper_link: geometry collision mesh filename=.//meshes/urdf/obj_combined_hulls/torso_pitch_upper_link.obj; visual mesh filename=.//meshes/urdf/obj_combined_hulls/torso_pitch_upper_link.obj
- link torso_yaw_link: geometry collision mesh filename=.//meshes/urdf/obj_combined_hulls/torso_yaw_link.obj; visual mesh filename=.//meshes/urdf/obj_combined_hulls/torso_yaw_link.obj
