Commit message: Condensed testing files into a single file, removed files no longer needed
Visualize_example and test_time were combined into a single file in which
user input determines what we are testing and the parameters neede.
Old example files were deleted while new ones were added, unneccessary URDF information
from the robot was deleted

File: test_arm/robot_obj_combined_hulls.urdf (robot description, URDF)
Before this commit: robot LSA, 17 links, 16 joints
Links:
- removed link right_dorsal_tracker_link
- removed link right_grip_point_link
- removed link right_haptx_dorsal_tracker_link
- removed link right_haptx_origin_tracker_link
Joints:
- removed joint right_dorsal_tracker
- removed joint right_grip_point
- removed joint right_haptx_dorsal_tracker
- removed joint right_haptx_origin_tracker

Commit message: Vectorized distance prediction functions in arm_test_time so they will run faster

File: test_arm/robot_obj_combined_hulls.urdf (robot description, URDF)
Before this commit: robot test_arm, 13 links, 12 joints
Links:
- link root_link: mass 7.183594348600132 -> None; geometry 
- link torso_pitch_lower_link: mass 0.5423763129502652 -> None; geometry 
- link torso_pitch_upper_link: mass 5.391439784540943 -> None; geometry 
- link torso_yaw_link: mass 1.922 -> None; geometry 
Joints:
- joint torso_pitch_lower: axis -3.059755751267585e-14 6.233280923648332e-14 1.0000000000000073 -> (none); limit lower=-0.5235987755982988 upper=0.2617993877991494 effort=70.0 velocity=4.1 -> (none); type revolute -> fixed
- joint torso_pitch_upper: axis -1.8748044307837196e-17 -3.013566795201047e-14 0.9999999999999998 -> (none); limit effort=70.0 velocity=4.1 -> (none); mimic joint=torso_pitch_lower multiplier=-1.0 offset=0 -> (none); type continuous -> fixed
- joint torso_yaw: axis 2.2135793071084816e-14 -3.77717399908133e-14 1.0000000000000007 -> (none); limit lower=-0.7853981633974483 upper=0.7853981633974483 effort=70.0 velocity=4.1 -> (none); type revolute -> fixed
